File: devboard.kicad_pcb (KiCad board)
At the start: 2 copper layers, 23 x 52 mm, 24 parts, among them J1 USB4105-GF-A, J2 Conn_01x08_Pin, J3 Conn_01x08_Pin, U1 STM32F411CEU6, U2 AP2120N-3.3TRG1, U3 USBLC6-2SC6Y

Commit message: Expose A13 to work with ST-Link
Parts:
- R5: value 330Ω -> 10k Ω
- moved C3 3.08 mm to (119.4, 99.8), turned to -90 degrees
- moved C2 1.51 mm to (118.3, 99.8), turned to -90 degrees
Connections:
- J3 pad 1: B8 -> B7
- J3 pad 2: B7 -> B6
- J3 pad 3: B6 -> B5
- J3 pad 4: B5 -> B4
- J3 pad 5: B4 -> B3
- J3 pad 6: B3 -> A15
- J3 pad 7: A15 -> A14
- J3 pad 8: A14 -> A13
Routing:
- net B8: track 17.8 -> 0.00 mm
- net A13: track 0.00 -> 10.4 mm
- net GND: track 26.6 -> 29.5 mm, vias 38 -> 36
- net +3.3V: track 95.9 -> 93.4 mm, vias 6 -> 5
- net B7: track 16.2 -> 18.7 mm
- net B6: track 14.2 -> 16.6 mm
- net B5: track 12.2 -> 14.6 mm
- net B4: track 10.2 -> 12.6 mm
- net B3: track 8.17 -> 10.5 mm
- net A15: track 6.76 -> 8.47 mm
- net A14: track 5.91 -> 6.97 mm
Other:
- board text added: "A13"
- board text removed: "B8"
